Commit message: Rename the folder basic_urdf_tutorial to r2d2_urdf_tutorial

File: r2d2_urdf_tutorial/urdf/05-visual.urdf (robot description, URDF)
Before this commit: robot visual, 16 links, 15 joints
Links:
- link left_gripper: geometry visual mesh filename=package://urdf_tutorial/meshes/l_finger.dae
- link left_tip: geometry visual mesh filename=package://urdf_tutorial/meshes/l_finger_tip.dae
- link right_gripper: geometry visual mesh filename=package://urdf_tutorial/meshes/l_finger.dae
- link right_tip: geometry visual mesh filename=package://urdf_tutorial/meshes/l_finger_tip.dae
Joints:
- joint gripper_extension: limit lower=-0.38 upper=0 effort=1000.0 velocity=0.5 -> (none); type prismatic -> fixed
- joint head_swivel: axis 0 0 1 -> (none); type continuous -> fixed
- joint left_back_wheel_joint: axis 0 1 0 -> (none); type continuous -> fixed
- joint left_front_wheel_joint: axis 0 1 0 -> (none); type continuous -> fixed
- joint left_gripper_joint: axis 0 0 1 -> (none); limit lower=0.0 upper=0.548 effort=1000.0 velocity=0.5 -> (none); type revolute -> fixed
- joint right_back_wheel_joint: axis 0 1 0 -> (none); type continuous -> fixed
- joint right_front_wheel_joint: axis 0 1 0 -> (none); type continuous -> fixed
- joint right_gripper_joint: axis 0 0 -1 -> (none); limit lower=0.0 upper=0.548 effort=1000.0 velocity=0.5 -> (none); type revolute -> fixed

File: r2d2_urdf_tutorial/urdf/06-flexible.urdf (robot description, URDF)
Before this commit: robot visual, 16 links, 15 joints
Links:
- link left_gripper: geometry visual mesh filename=package://urdf_tutorial/meshes/l_finger.dae
- link left_tip: geometry visual mesh filename=package://urdf_tutorial/meshes/l_finger_tip.dae
- link right_gripper: geometry visual mesh filename=package://urdf_tutorial/meshes/l_finger.dae
- link right_tip: geometry visual mesh filename=package://urdf_tutorial/meshes/l_finger_tip.dae
Joints:
- joint gripper_extension: limit (none) -> lower=-0.38 upper=0 effort=1000.0 velocity=0.5; type fixed -> prismatic
- joint head_swivel: axis (none) -> 0 0 1; type fixed -> continuous
- joint left_back_wheel_joint: axis (none) -> 0 1 0; type fixed -> continuous
- joint left_front_wheel_joint: axis (none) -> 0 1 0; type fixed -> continuous
- joint left_gripper_joint: axis (none) -> 0 0 1; limit (none) -> lower=0.0 upper=0.548 effort=1000.0 velocity=0.5; type fixed -> revolute
- joint right_back_wheel_joint: axis (none) -> 0 1 0; type fixed -> continuous
- joint right_front_wheel_joint: axis (none) -> 0 1 0; type fixed -> continuous
- joint right_gripper_joint: axis (none) -> 0 0 -1; limit (none) -> lower=0.0 upper=0.548 effort=1000.0 velocity=0.5; type fixed -> revolute

File: r2d2_urdf_tutorial/urdf/09-roscontrol.urdf.xacro (robot description, xacro)
@@ -1,4 +1,4 @@
 <?xml version="1.0"?>
-<robot name="macroed" xmlns:xacro="http://ros.org/wiki/xacro">
+<robot name="roscontrol" xmlns:xacro="http://ros.org/wiki/xacro">
   <xacro:property name="width" value="0.2" />
   <xacro:property name="leglen" value="0.6" />
@@ -60,4 +60,24 @@
       <origin xyz="${baselen*reflect/3} 0 -${wheeldiam/2+.05}" rpy="0 0 0"/>
     </joint>
+    <!-- This block provides the simulator (Gazebo) with information on a few additional
+    physical properties. See http://gazebosim.org/tutorials/?tut=ros_urdf for more-->
+    <gazebo reference="${prefix}_${suffix}_wheel">
+      <mu1 value="200.0"/>
+      <mu2 value="100.0"/>
+      <kp value="10000000.0" />
+      <kd value="1.0" />
+      <material>Gazebo/Grey</material>
+    </gazebo>
+    <!-- This block connects the wheel joint to an actuator (motor), which informs both
+    simulation and visualization of the robot -->
+    <transmission name="${prefix}_${suffix}_wheel_trans">
+      <type>transmission_interface/SimpleTransmission</type>
+      <actuator name="${prefix}_${suffix}_wheel_motor">
+        <mechanicalReduction>1</mechanicalReduction>
+      </actuator>
+      <joint name="${prefix}_${suffix}_wheel_joint">
+        <hardwareInterface>VelocityJointInterface</hardwareInterface>
+      </joint>
+    </transmission>
   </xacro:macro>
   <xacro:macro name="leg" params="prefix reflect">
@@ -112,4 +132,6 @@
     <limit effort="1000.0" lower="-${width*2-.02}" upper="0" velocity="0.5"/>
     <origin rpy="0 0 0" xyz="${width-.01} 0 0.2"/>
+    <limit effort="30" velocity="0.2"/>
+    <dynamics damping="0.0" friction="0.0"/>
   </joint>
   <link name="gripper_pole">
@@ -128,4 +150,13 @@
     <xacro:default_inertial mass="0.05"/>
   </link>
+  <transmission name="gripper_extension_trans">
+    <type>transmission_interface/SimpleTransmission</type>
+    <actuator name="gripper_extension_motor">
+      <mechanicalReduction>1</mechanicalReduction>
+    </actuator>
+    <joint name="gripper_extension">
+      <hardwareInterface>PositionJointInterface</hardwareInterface>
+    </joint>
+  </transmission>
   <xacro:macro name="gripper" params="prefix reflect">
     <joint name="${prefix}_gripper_joint" type="revolute">
@@ -135,4 +166,6 @@
       <parent link="gripper_pole"/>
       <child link="${prefix}_gripper"/>
+      <limit effort="30" velocity="1.0"/>
+      <dynamics damping="0.0" friction="0.0"/>
     </joint>
     <link name="${prefix}_gripper">
@@ -151,4 +184,13 @@
       <xacro:default_inertial mass="0.05"/>
     </link>
+    <transmission name="${prefix}_gripper_trans">
+      <type>transmission_interface/SimpleTransmission</type>
+      <actuator name="${prefix}_gripper_motor">
+        <mechanicalReduction>1</mechanicalReduction>
+      </actuator>
+      <joint name="${prefix}_gripper_joint">
+        <hardwareInterface>PositionJointInterface</hardwareInterface>
+      </joint>
+    </transmission>
     <joint name="${prefix}_tip_joint" type="fixed">
       <parent link="${prefix}_gripper"/>
@@ -193,5 +235,8 @@
     <origin xyz="0 0 ${bodylen/2}"/>
     <limit effort="30" velocity="1.0"/>
+    <dynamics damping="0.0" friction="0.0"/>
   </joint>
+  <!-- This block connects the head_swivel joint to an actuator (motor), which informs both
+  simulation and visualization of the robot -->
   <transmission name="head_swivel_trans">
     <type>transmission_interface/SimpleTransmission</type>
@@ -223,4 +268,5 @@
     <origin xyz="${.707*width+0.04} 0 ${.707*width}"/>
   </joint>
+  <!-- Gazebo plugin for ROS Control -->
   <gazebo>
     <plugin name="gazebo_ros_control" filename="libgazebo_ros_control.so">
